Commit message: second push

File: Collision_Avoidance/d435/tools/d435.gazebo.xacro (robot description, xacro)
@@ -21,5 +21,5 @@
       <plugin name="camera_controller" filename="libgazebo_ros_camera.so">
         <alwaysOn>true</alwaysOn>
-        <updateRate>30.0</updateRate>
+        <updateRate>30</updateRate>
         <cameraName>camera</cameraName>
         <frameName>camera_color_optical_frame</frameName>
@@ -168,7 +168,8 @@
         <height>480</height>
         <format>L_INT8</format>
+        <!-- <format>L8</format> -->
       </image>
       <clip>
-        <near>0</near>
+        <near>0.105</near>
         <far>10</far>
       </clip>
@@ -185,6 +186,6 @@
           <pointCloudTopicName>/ir_depth/depth/points</pointCloudTopicName>
           <frameName>ir_depth</frameName>
-          <pointCloudCutoff>0.5</pointCloudCutoff>
-          <pointCloudCutoffMax>3.0</pointCloudCutoffMax>
+          <pointCloudCutoff>0.1</pointCloudCutoff>
+          <pointCloudCutoffMax>10</pointCloudCutoffMax>
           <distortionK1>0</distortionK1>
           <distortionK2>0</distortionK2>

File: Collision_Avoidance/wrs_gazebo/mobile_dual_arm/urdf/mobile_dual_arm.xacro (robot description, xacro)
@@ -12,4 +12,5 @@
   <!-- <link name="base_link" /> -->
   <xacro:realsense_d435 connected_to="world" complett_links="true" ns="0" xyz="-0.05 0 1.8" rpy = "0 1 0"/>
+  <!-- <xacro:realsense_d435 connected_to="world" complett_links="true" ns="0" xyz="-0.05 0 1.8" rpy = "0 0.85 0"/> -->
   <!-- <xacro:realsense_d435 connected_to="world" complett_links="true" ns="1" xyz="0.01 0 1.3" rpy = "0 0 0"/> -->
   <!-- <joint name="fixed1" type="fixed">
@@ -39,15 +40,4 @@
     <origin xyz="0 0.016 0" rpy="0 0 1.57" />
   </xacro:suction>
-  <!-- <joint name="fixed4" type="fixed">
-    <origin
-      xyz="0 0 0.562"
-      rpy="0 0 0" />
-    <parent link="world"/>
-    <child link="base_link"/>
-  </joint> -->
-<!--
-  <xacro:realsense_d435 connected_to="base_link" complett_links="true" ns="" xyz="0.01 0 5" rpy = "0 0 0">
-    <origin xyz="0 0.016 0" rpy="0 0 1.57" />
-  </xacro:realsense_d435> -->
   <!--joint name="fixed" type="fixed">
     <origin
